Commit message: The launch file runs without major errors
I think from here I can make a little readme explaining how to create
the numsr_franka_moveit_config package, and how to include the franka
packages, maybe using vcs?

Now i need to figure out why none of my services work?

File: franka_teleop/config/hand.xacro (robot description, xacro)
@@ -13,5 +13,5 @@
       <visual>
         <geometry>
-          <mesh filename="package://franka_description/meshes/visual/hand.dae"/>
+          <mesh filename="package://franka_teleop/meshes/visual/hand.dae"/>
         </geometry>
       </visual>
@@ -63,5 +63,5 @@
       <visual>
         <geometry>
-          <mesh filename="package://franka_description/meshes/visual/finger.dae"/>
+          <mesh filename="package://franka_teleop/meshes/visual/finger.dae"/>
         </geometry>
       </visual>
@@ -71,5 +71,5 @@
         <origin xyz="0 0 0" rpy="0 0 ${pi}"/>
         <geometry>
-          <mesh filename="package://franka_description/meshes/visual/finger.dae"/>
+          <mesh filename="package://franka_teleop/meshes/visual/finger.dae"/>
         </geometry>
       </visual>

File: franka_teleop/config/panda_arm.urdf (robot description, URDF)
Before this commit: robot panda, 13 links, 12 joints
Links:
- link panda_hand: geometry collision cylinder length=0.1 radius=0.05; collision cylinder length=0.1 radius=0.07
- link panda_leftfinger: geometry visual mesh filename=package://franka_teleop/meshes/visual/finger.dae
- link panda_rightfinger: geometry visual mesh filename=package://franka_teleop/meshes/visual/finger.dae

File: numsr_franka_moveit_config/config/panda.urdf.xacro (robot description, xacro)
@@ -5,5 +5,6 @@
     <xacro:include filename="panda_arm.urdf" />
     <!-- Import control_xacro -->
-    <xacro:include filename="panda.ros2_control.xacro" />
-    <xacro:panda_ros2_control name="FakeSystem" initial_positions_file="$(arg initial_positions_file)"/>
+    <!-- I edited this file by hand! -->
+    <xacro:include filename="$(find franka_description)/robots/panda_arm.ros2_control.xacro" />
+    <!-- <xacro:panda_ros2_control name="FakeSystem" initial_positions_file="$(arg initial_positions_file)"/> -->
 </robot>
