Commit message: Deleted some unnecessary files
Also changed the name of the moveit package to numsr_franka_moveit_config

Am going to remove some unnecessary direcotries inside franka_teleop next,
so I want to save my place in case those directories turn out to be
necessary

File: numsr_franka_moveit_config/config/panda.urdf.xacro (robot description, xacro)
@@ -3,5 +3,5 @@
     <xacro:arg name="initial_positions_file" default="initial_positions.yaml" />
     <!-- Import panda urdf file -->
-    <xacro:include filename="$(find franka_teleop)/config/panda_arm.urdf" />
+    <xacro:include filename="panda_arm.urdf" />
     <!-- Import control_xacro -->
     <xacro:include filename="panda.ros2_control.xacro" />

File: numsr_franka_moveit_config/config/panda_arm.urdf (robot description, URDF)
Before this commit: robot panda, 13 links, 12 joints
Links:
- link panda_hand: geometry collision cylinder length=0.1 radius=0.05; collision cylinder length=0.1 radius=0.07
- link panda_leftfinger: geometry visual mesh filename=package://msr_franka_moveit_config/meshes/visual/finger.dae
- link panda_link0: geometry collision cylinder length=0.03 radius=0.09; collision sphere radius=0.09
- link panda_link1: geometry collision cylinder length=0.2830 radius=0.09; collision sphere radius=0.09
- link panda_link2: geometry collision cylinder length=0.12 radius=0.09; collision sphere radius=0.09
- link panda_link3: geometry collision cylinder length=0.15 radius=0.09; collision sphere radius=0.09
- link panda_link4: geometry collision cylinder length=0.12 radius=0.09; collision sphere radius=0.09
- link panda_link5: geometry collision cylinder length=0.1 radius=0.09; collision cylinder length=0.14 radius=0.055
- link panda_link6: geometry collision cylinder length=0.08 radius=0.08; collision sphere radius=0.08
- link panda_link7: geometry collision cylinder length=0.14 radius=0.07; collision sphere radius=0.07
- link panda_rightfinger: geometry visual mesh filename=package://msr_franka_moveit_config/meshes/visual/finger.dae

Commit message: This is the first version to successfully plan

File: numsr_franka_moveit_config/config/panda.urdf.xacro (robot description, xacro)
@@ -6,5 +6,5 @@
     <!-- Import control_xacro -->
     <!-- I edited this file by hand! -->
-    <xacro:include filename="$(find franka_description)/robots/panda_arm.ros2_control.xacro" />
+    <xacro:include filename="$(find numsr_franka_moveit_config)/config/panda_arm.ros2_control.xacro" />
     <!-- <xacro:panda_ros2_control name="FakeSystem" initial_positions_file="$(arg initial_positions_file)"/> -->
 </robot>

File: numsr_franka_moveit_config/config/panda_arm.urdf (robot description, URDF)
Before this commit: robot panda, 13 links, 12 joints
Joints:
- joint panda_joint8: origin xyz=0 0 0.107 rpy=0 0 0 -> xyz=0 0 0.107 rpy=0 0 -0.7853981633974483
