Commit message: Can plan paths and execute them accurately
I now know how to plan and execute a path to a point based on a point in
space and a quaternion. I should write some extra functions for planning
based on specific joint positions, and also a function for planning and
executing sequentially without having to make two service calls.

File: numsr_franka_moveit_config/config/panda_arm.urdf (robot description, URDF)
Before this commit: robot panda, 13 links, 12 joints
Joints:
- joint panda_joint8: origin xyz=0 0 0.107 rpy=0 0 -0.7853981633974483 -> xyz=0 0 0.107 rpy=0 0 0
