Commit message: state of code for the final demo on 3/15
Very slight modifications were made to the code, mainly adjusting PD
values and force thresholds. I never was able to control the force
applied by the gripper on arbitrary objects, or any objects for that
matter. This is something that I really want to figure out in the
future. I also need to one day switch over to the
PandaJointGroupController, I think it was called that. Apparently this
is the actual controller many people use for servoing the franka, UR5
and other robots, but I didn't know about that until today. I also want
to implement my own bounding box so I don't get any weird behavior when
approaching joint limits of the robot.

File: numsr_franka_moveit_config/config/panda_arm_real.urdf (robot description, URDF)
Before this commit: robot panda, 13 links, 12 joints
Joints:
- joint panda_finger_joint1: limit lower=0.0 upper=0.04 effort=20 velocity=0.2 -> lower=0.0 upper=0.04 effort=1.0 velocity=0.2
- joint panda_finger_joint2: limit lower=0.0 upper=0.04 effort=20 velocity=0.2 -> lower=0.0 upper=0.04 effort=1.0 velocity=0.2
